File: HW/picoMacro/picoMacro.sch (KiCad schematic (older format))
At the start: 53 parts, among them SW1 SW_Push, SW10 SW_Push, SW11 SW_Push, SW12 SW_Push, SW13 SW_Push, SW14 SW_Push, SW15 SW_Push, SW16 SW_Push, SW2 SW_Push, SW3 SW_Push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

Commit message: added description of the key shortcut storage method
Parts:
- C17, C18: symbol Device:CP -> picoMacro-rescue:CP-Device
- Disp1: symbol DisplayCustom:1.3_OLED_SH1106 -> picoMacro-rescue:1.3_OLED_SH1106-DisplayCustom
- LED1, LED10, LED11, LED12, LED13, LED14, LED15, LED16, LED2, LED3, LED4, LED5, LED6, LED7, LED8, LED9: symbol WS2812-2020:WS2812-2020 -> picoMacro-rescue:WS2812-2020-WS2812-2020
- U1: symbol MCU_RaspberryPi_and_Boards:Pico -> picoMacro-rescue:Pico-MCU_RaspberryPi_and_Boards
